File: prawnblaster_pcb.kicad_sch (KiCad schematic)
At the start: 30 parts, among them J1 USB_B, J2 Conn_01x04, J3 Conn_Coaxial_x2, J4 Conn_Coaxial_x2, J5 Conn_Coaxial, J6 Conn_Coaxial, J7 Conn_01x02, U1 Pico, U2 ADuM5000, U3 ADUM4160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

Commit message: Fixed trigger plug wiring
Parts:
- removed J3, J4: Conn_Coaxial_x2, Connector_Coaxial:BNC_Amphenol_031-6575_Horizontal, symbol Connector:Conn_Coaxial_x2
- added J3: Clock01, Connector_Coaxial:BNC_Amphenol_031-6575_Horizontal, symbol Connector:Conn_Coaxial_x2_Isolated
- added J4: Clock23, Connector_Coaxial:BNC_Amphenol_031-6575_Horizontal, symbol Connector:Conn_Coaxial_x2_Isolated
Connections:
- net GND: now also J3.2 (Ext1), J3.4 (Ext2), J4.2 (Ext1), J4.4 (Ext2)
- net at U4.11 (B7), U4.12 (B6): now also J3.1 (In1)
- net at U4.13 (B5), U4.14 (B4): now also J3.3 (In2)
- net at U4.15 (B3), U4.16 (B2): now also J4.1 (In1)
- net at U4.17 (B1), U4.18 (B0): now also J4.3 (In2)
